File: Schematic/usermoves.sch (KiCad schematic (older format))
At the start: 54 parts, among them SW1 SW_Push, SW2 SW_Push, SW3 SW_Push, SW4 SW_Push, SW5 SW_Push, SW6 SW_Push, SW7 SW_Push, SW8 SW_Push, SW9 SW_Push, U1 74LS107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

Commit message: More work on the circuit and the PCB layout.
Parts:
- removed R13, R15, R20, R22, R24: 10K, Resistor_THT:R_Axial_DIN0204_L3.6mm_D1.6mm_P1.90mm_Vertical, symbol ttt_ttl-rescue:R_Small
- removed R14, R19, R21, R23: 1K, Resistor_THT:R_Axial_DIN0204_L3.6mm_D1.6mm_P1.90mm_Vertical, symbol ttt_ttl-rescue:R_Small
- R11, R2, R4, R6: value 10K -> 1K
- U1, U2, U3, U4, U5, U6, U7, U8, U9: value 74LS107 -> 74LS109
Connections:
- wire segments 153 -> 144
Other:
- moved on the sheet: R3, SW2

Commit message: Fixed up the reset line circuitry
Parts:
- R16, R17, R18, R25, R26, R27, R7, R8, R9: value 10K -> 1K
Changed lines of the file:
@@
 P 3300 850
 F 0 "R7" V 3200 900 50  0000 L CNN
-F 1 "10K" V 3200 700 50  0000 L CNN
+F 1 "1K" V 3200 700 50  0000 L CNN
 F 2 "Resistor_THT:R_Axial_DIN0204_L3.6mm_D1.6mm_P1.90mm_Vertical" H 3300 850 50  0001 C CNN
 F 3 "" H 3300 850 50  0001 C CNN
@@
 P 7000 850
 F 0 "R16" V 6900 900 50  0000 L CNN
-F 1 "10K" V 6900 700 50  0000 L CNN
+F 1 "1K" V 6900 700 50  0000 L CNN
 F 2 "Resistor_THT:R_Axial_DIN0204_L3.6mm_D1.6mm_P1.90mm_Vertical" H 7000 850 50  0001 C CNN
 F 3 "" H 7000 850 50  0001 C CNN
@@
 P 10550 850
 F 0 "R25" V 10450 900 50  0000 L CNN
-F 1 "10K" V 10450 700 50  0000 L CNN
+F 1 "1K" V 10450 700 50  0000 L CNN
 F 2 "Resistor_THT:R_Axial_DIN0204_L3.6mm_D1.6mm_P1.90mm_Vertical" H 10550 850 50  0001 C CNN
 F 3 "" H 10550 850 50  0001 C CNN
@@
 P 3350 2900
 F 0 "R8" V 3250 2950 50  0000 L CNN
-F 1 "10K" V 3250 2750 50  0000 L CNN
+F 1 "1K" V 3250 2750 50  0000 L CNN
 F 2 "Resistor_THT:R_Axial_DIN0204_L3.6mm_D1.6mm_P1.90mm_Vertical" H 3350 2900 50  0001 C CNN
 F 3 "" H 3350 2900 50  0001 C CNN
@@
 P 7050 2900
 F 0 "R17" V 6950 2950 50  0000 L CNN
-F 1 "10K" V 6950 2750 50  0000 L CNN
+F 1 "1K" V 6950 2750 50  0000 L CNN
 F 2 "Resistor_THT:R_Axial_DIN0204_L3.6mm_D1.6mm_P1.90mm_Vertical" H 7050 2900 50  0001 C CNN
 F 3 "" H 7050 2900 50  0001 C CNN
@@
 P 10600 2900
 F 0 "R26" V 10500 2950 50  0000 L CNN
-F 1 "10K" V 10500 2750 50  0000 L CNN
+F 1 "1K" V 10500 2750 50  0000 L CNN
 F 2 "Resistor_THT:R_Axial_DIN0204_L3.6mm_D1.6mm_P1.90mm_Vertical" H 10600 2900 50  0001 C CNN
 F 3 "" H 10600 2900 50  0001 C CNN
@@
 P 3350 4800
 F 0 "R9" V 3250 4850 50  0000 L CNN
-F 1 "10K" V 3250 4650 50  0000 L CNN
+F 1 "1K" V 3250 4650 50  0000 L CNN
 F 2 "Resistor_THT:R_Axial_DIN0204_L3.6mm_D1.6mm_P1.90mm_Vertical" H 3350 4800 50  0001 C CNN
 F 3 "" H 3350 4800 50  0001 C CNN
@@
 P 7050 4800
 F 0 "R18" V 6950 4850 50  0000 L CNN
-F 1 "10K" V 6950 4650 50  0000 L CNN
+F 1 "1K" V 6950 4650 50  0000 L CNN
 F 2 "Resistor_THT:R_Axial_DIN0204_L3.6mm_D1.6mm_P1.90mm_Vertical" H 7050 4800 50  0001 C CNN
 F 3 "" H 7050 4800 50  0001 C CNN
@@
 P 10600 4800
 F 0 "R27" V 10500 4850 50  0000 L CNN
-F 1 "10K" V 10500 4650 50  0000 L CNN
+F 1 "1K" V 10500 4650 50  0000 L CNN
 F 2 "Resistor_THT:R_Axial_DIN0204_L3.6mm_D1.6mm_P1.90mm_Vertical" H 10600 4800 50  0001 C CNN
 F 3 "" H 10600 4800 50  0001 C CNN

Commit message: Updated the schematic and PCB with the new flip-flip pinouts and footprints.
Parts:
- U1, U2, U3, U4, U5, U6, U7, U8, U9: footprint Package_DIP:DIP-14_W7.62mm -> Package_DIP:DIP-16_W7.62mm; symbol ttt_ttl-rescue:74LS107 -> local:74LS107
Connections:
- net labels added: Move1, Move2, Move3, Move4, Move5, Move6, Move7, Move8, Move9
- net labels removed: Board1, Board2, Board3, Board4, Board5, Board6, Board7, Board8, Board9
- wire segments 144 -> 162
Changed lines of the file:
@@
 $EndDescr
 $Comp
-L ttt_ttl-rescue:74LS107 U1
+L local:74LS107 U1
 U 1 1 5CF7BC39
 P 2450 1550
 F 0 "U1" H 2450 1650 50  0000 C CNN
 F 1 "74LS109" H 2450 1450 50  0000 C CNN
-F 2 "Package_DIP:DIP-14_W7.62mm" H 2450 1550 50  0001 C CNN
+F 2 "Package_DIP:DIP-16_W7.62mm" H 2450 1550 50  0001 C CNN
 F 3 "" H 2450 1550 50  0001 C CNN
 	1    2450 1550
@@
 	2350 2250 2450 2250
 Text GLabel 1700 1800 0    60   Input ~ 0
-Board1
+Move1
 Wire Wire Line
 	1700 1800 1800 1800
@@
 	3150 850  3150 950
 $Comp
-L ttt_ttl-rescue:74LS107 U2
+L local:74LS107 U2
 U 1 1 5CF7BC3C
 P 6150 1550
 F 0 "U2" H 6150 1650 50  0000 C CNN
 F 1 "74LS109" H 6150 1450 50  0000 C CNN
-F 2 "Package_DIP:DIP-14_W7.62mm" H 6150 1550 50  0001 C CNN
+F 2 "Package_DIP:DIP-16_W7.62mm" H 6150 1550 50  0001 C CNN
 F 3 "" H 6150 1550 50  0001 C CNN
 	1    6150 1550
@@
 	6050 2250 6150 2250
 Text GLabel 5400 1800 0    60   Input ~ 0
-Board2
+Move2
 Wire Wire Line
 	5400 1800 5500 1800
@@
 	9600 2250 9700 2250
 Text GLabel 8950 1800 0    60   Input ~ 0
-Board3
+Move3
 Wire Wire Line
 	8950 1800 9050 1800
@@
 	10400 850  10400 950
 $Comp
-L ttt_ttl-rescue:74LS107 U4
+L local:74LS107 U4
 U 1 1 5CF7BC42
 P 2500 3600
 F 0 "U4" H 2500 3700 50  0000 C CNN
 F 1 "74LS109" H 2500 3500 50  0000 C CNN
-F 2 "Package_DIP:DIP-14_W7.62mm" H 2500 3600 50  0001 C CNN
+F 2 "Package_DIP:DIP-16_W7.62mm" H 2500 3600 50  0001 C CNN
 F 3 "" H 2500 3600 50  0001 C CNN
 	1    2500 3600
@@
 	2400 4300 2500 4300
 Text GLabel 1750 3850 0    60   Input ~ 0
-Board4
+Move4
 Wire Wire Line
 	1750 3850 1850 3850
@@
 	3200 2900 3200 3000
 $Comp
-L ttt_ttl-rescue:74LS107 U5
+L local:74LS107 U5
 U 1 1 5CF7BC45
 P 6200 3600
 F 0 "U5" H 6200 3700 50  0000 C CNN
 F 1 "74LS109" H 6200 3500 50  0000 C CNN
-F 2 "Package_DIP:DIP-14_W7.62mm" H 6200 3600 50  0001 C CNN
+F 2 "Package_DIP:DIP-16_W7.62mm" H 6200 3600 50  0001 C CNN
 F 3 "" H 6200 3600 50  0001 C CNN
 	1    6200 3600
@@
 	6100 4300 6200 4300
 Text GLabel 5450 3850 0    60   Input ~ 0
-Board5
+Move5
 Wire Wire Line
 	5450 3850 5550 3850
@@
 	6900 2900 6900 3000
 $Comp
-L ttt_ttl-rescue:74LS107 U6
+L local:74LS107 U6
 U 1 1 5CF7B1B2
 P 9750 3600
 F 0 "U6" H 9750 3700 50  0000 C CNN
 F 1 "74LS109" H 9750 3500 50  0000 C CNN
-F 2 "Package_DIP:DIP-14_W7.62mm" H 9750 3600 50  0001 C CNN
+F 2 "Package_DIP:DIP-16_W7.62mm" H 9750 3600 50  0001 C CNN
 F 3 "" H 9750 3600 50  0001 C CNN
 	1    9750 3600
@@
 	9650 4300 9750 4300
 Text GLabel 9000 3850 0    60   Input ~ 0
-Board6
+Move6
 Wire Wire Line
 	9000 3850 9100 3850
@@
 	10450 2900 10450 3000
 $Comp
-L ttt_ttl-rescue:74LS107 U7
+L local:74LS107 U7
 U 1 1 5CF7BC4B
 P 2500 5500
 F 0 "U7" H 2500 5600 50  0000 C CNN
 F 1 "74LS109" H 2500 5400 50  0000 C CNN
-F 2 "Package_DIP:DIP-14_W7.62mm" H 2500 5500 50  0001 C CNN
+F 2 "Package_DIP:DIP-16_W7.62mm" H 2500 5500 50  0001 C CNN
 F 3 "" H 2500 5500 50  0001 C CNN
 	1    2500 5500
@@
 	2400 6200 2500 6200
 Text GLabel 1750 5750 0    60   Input ~ 0
-Board7
+Move7
 Wire Wire Line
 	1750 5750 1850 5750
@@
 	3200 4800 3200 4900
 $Comp
-L ttt_ttl-rescue:74LS107 U8
+L local:74LS107 U8
 U 1 1 5CF7B8A4
 P 6200 5500
 F 0 "U8" H 6200 5600 50  0000 C CNN
 F 1 "74LS109" H 6200 5400 50  0000 C CNN
-F 2 "Package_DIP:DIP-14_W7.62mm" H 6200 5500 50  0001 C CNN
+F 2 "Package_DIP:DIP-16_W7.62mm" H 6200 5500 50  0001 C CNN
 F 3 "" H 6200 5500 50  0001 C CNN
 	1    6200 5500
@@
 	6100 6200 6200 6200
 Text GLabel 5450 5750 0    60   Input ~ 0
-Board8
+Move8
 Wire Wire Line
 	5450 5750 5550 5750
@@
 	6900 4800 6900 4900
 $Comp
-L ttt_ttl-rescue:74LS107 U9
+L local:74LS107 U9
 U 1 1 5CF7B8E1
 P 9750 5500
 F 0 "U9" H 9750 5600 50  0000 C CNN
 F 1 "74LS109" H 9750 5400 50  0000 C CNN
-F 2 "Package_DIP:DIP-14_W7.62mm" H 9750 5500 50  0001 C CNN
+F 2 "Package_DIP:DIP-16_W7.62mm" H 9750 5500 50  0001 C CNN
 F 3 "" H 9750 5500 50  0001 C CNN
 	1    9750 5500
@@
 	9650 6200 9750 6200
 Text GLabel 9000 5750 0    60   Input ~ 0
-Board9
+Move9
 Wire Wire Line
 	9000 5750 9100 5750
@@
 	8500 3650 8500 3700
 $Comp
-L ttt_ttl-rescue:74LS107 U3
+L local:74LS107 U3
 U 1 1 5CF7BC3F
 P 9700 1550
 F 0 "U3" H 9700 1650 50  0000 C CNN
 F 1 "74LS109" H 9700 1450 50  0000 C CNN
-F 2 "Package_DIP:DIP-14_W7.62mm" H 9700 1550 50  0001 C CNN
+F 2 "Package_DIP:DIP-16_W7.62mm" H 9700 1550 50  0001 C CNN
 F 3 "" H 9700 1550 50  0001 C CNN
 	1    9700 1550
@@
 Wire Wire Line
 	8500 5550 8500 5600
+Text GLabel 2300 800  0    60   Input ~ 0
+Hi
+Wire Wire Line
+	2450 950  2450 800
+Wire Wire Line
+	2450 800  2300 800
+Text GLabel 9550 4750 0    60   Input ~ 0
+Hi
+Wire Wire Line
+	9750 4900 9750 4750
+Wire Wire Line
+	9750 4750 9550 4750
+Text GLabel 6000 4750 0    60   Input ~ 0
+Hi
+Wire Wire Line
+	6200 4900 6200 4750
+Wire Wire Line
+	6200 4750 6000 4750
+Text GLabel 2300 4750 0    60   Input ~ 0
+Hi
+Wire Wire Line
+	2500 4900 2500 4750
+Wire Wire Line
+	2500 4750 2300 4750
+Text GLabel 2350 2850 0    60   Input ~ 0
+Hi
+Wire Wire Line
+	2500 3000 2500 2850
+Wire Wire Line
+	2500 2850 2350 2850
+Text GLabel 6050 2850 0    60   Input ~ 0
+Hi
+Wire Wire Line
+	6200 3000 6200 2850
+Wire Wire Line
+	6200 2850 6050 2850
+Text GLabel 9500 2850 0    60   Input ~ 0
+Hi
+Wire Wire Line
+	9750 3000 9750 2850
+Wire Wire Line
+	9750 2850 9500 2850
+Text GLabel 9550 850  0    60   Input ~ 0
+Hi
+Wire Wire Line
+	9700 950  9700 850
+Wire Wire Line
+	9700 850  9550 850
+Text GLabel 6000 800  0    60   Input ~ 0
+Hi
+Wire Wire Line
+	6150 950  6150 800
+Wire Wire Line
+	6150 800  6000 800
 $EndSCHEMATC

Commit message: Smaller 8Kx8 EEPROM is working
I managed to get the code to generate a ROM file which uses a 4-bit board
state plus the user's moves to look up the net board move and the next
board state. I've redone the schematic, PCB and I've started on the
documentation. I need to redraw the design diagram.
Parts:
- D1, D2, D3, D4, D5, D6, D7, D8, D9: footprint Diode_THT:D_DO-41_SOD81_P7.62mm_Horizontal -> LED_THT:LED_D3.0mm
Changed lines of the file:
@@
 F 0 "D1" V 3250 1100 50  0000 L CNN
 F 1 "LED" V 3150 1150 50  0000 L CNN
-F 2 "Diode_THT:D_DO-41_SOD81_P7.62mm_Horizontal" V 3150 1050 50  0001 C CNN
+F 2 "LED_THT:LED_D3.0mm" V 3150 1050 50  0001 C CNN
 F 3 "" V 3150 1050 50  0001 C CNN
 	1    3150 1050
@@
 F 0 "D4" V 6950 1100 50  0000 L CNN
 F 1 "LED" V 6850 1150 50  0000 L CNN
-F 2 "Diode_THT:D_DO-41_SOD81_P7.62mm_Horizontal" V 6850 1050 50  0001 C CNN
+F 2 "LED_THT:LED_D3.0mm" V 6850 1050 50  0001 C CNN
 F 3 "" V 6850 1050 50  0001 C CNN
 	1    6850 1050
@@
 F 0 "D7" V 10500 1100 50  0000 L CNN
 F 1 "LED" V 10400 1150 50  0000 L CNN
-F 2 "Diode_THT:D_DO-41_SOD81_P7.62mm_Horizontal" V 10400 1050 50  0001 C CNN
+F 2 "LED_THT:LED_D3.0mm" V 10400 1050 50  0001 C CNN
 F 3 "" V 10400 1050 50  0001 C CNN
 	1    10400 1050
@@
 F 0 "D2" V 3300 3150 50  0000 L CNN
 F 1 "LED" V 3200 3200 50  0000 L CNN
-F 2 "Diode_THT:D_DO-41_SOD81_P7.62mm_Horizontal" V 3200 3100 50  0001 C CNN
+F 2 "LED_THT:LED_D3.0mm" V 3200 3100 50  0001 C CNN
 F 3 "" V 3200 3100 50  0001 C CNN
 	1    3200 3100
@@
 F 0 "D5" V 7000 3150 50  0000 L CNN
 F 1 "LED" V 6900 3200 50  0000 L CNN
-F 2 "Diode_THT:D_DO-41_SOD81_P7.62mm_Horizontal" V 6900 3100 50  0001 C CNN
+F 2 "LED_THT:LED_D3.0mm" V 6900 3100 50  0001 C CNN
 F 3 "" V 6900 3100 50  0001 C CNN
 	1    6900 3100
@@
 F 0 "D8" V 10550 3150 50  0000 L CNN
 F 1 "LED" V 10450 3200 50  0000 L CNN
-F 2 "Diode_THT:D_DO-41_SOD81_P7.62mm_Horizontal" V 10450 3100 50  0001 C CNN
+F 2 "LED_THT:LED_D3.0mm" V 10450 3100 50  0001 C CNN
 F 3 "" V 10450 3100 50  0001 C CNN
 	1    10450 3100
@@
 F 0 "D3" V 3300 5050 50  0000 L CNN
 F 1 "LED" V 3200 5100 50  0000 L CNN
-F 2 "Diode_THT:D_DO-41_SOD81_P7.62mm_Horizontal" V 3200 5000 50  0001 C CNN
+F 2 "LED_THT:LED_D3.0mm" V 3200 5000 50  0001 C CNN
 F 3 "" V 3200 5000 50  0001 C CNN
 	1    3200 5000
@@
 F 0 "D6" V 7000 5050 50  0000 L CNN
 F 1 "LED" V 6900 5100 50  0000 L CNN
-F 2 "Diode_THT:D_DO-41_SOD81_P7.62mm_Horizontal" V 6900 5000 50  0001 C CNN
+F 2 "LED_THT:LED_D3.0mm" V 6900 5000 50  0001 C CNN
 F 3 "" V 6900 5000 50  0001 C CNN
 	1    6900 5000
@@
 F 0 "D9" V 10550 5050 50  0000 L CNN
 F 1 "LED" V 10450 5100 50  0000 L CNN
-F 2 "Diode_THT:D_DO-41_SOD81_P7.62mm_Horizontal" V 10450 5000 50  0001 C CNN
+F 2 "LED_THT:LED_D3.0mm" V 10450 5000 50  0001 C CNN
 F 3 "" V 10450 5000 50  0001 C CNN
 	1    10450 5000

Commit message: I bought different pushbuttons, so I updated the PCB design.
Parts:
- SW1, SW2, SW3, SW4, SW5, SW6, SW7, SW8, SW9: footprint Button_Switch_THT:SW_PUSH_6mm_H8mm -> Button_Switch_THT:Push_E-Switch_KS01Q01
Changed lines of the file:
@@
 F 0 "SW2" V 1200 3200 50  0000 L CNN
 F 1 "SW_Push" V 1100 3350 50  0000 C CNN
-F 2 "Button_Switch_THT:SW_PUSH_6mm_H8mm" H 1250 3300 50  0001 C CNN
+F 2 "Button_Switch_THT:Push_E-Switch_KS01Q01" H 1250 3300 50  0001 C CNN
 F 3 "" H 1250 3300 50  0001 C CNN
 	1    1250 3100
@@
 F 0 "SW4" V 4800 3200 50  0000 L CNN
 F 1 "SW_Push" V 4700 3350 50  0000 C CNN
-F 2 "Button_Switch_THT:SW_PUSH_6mm_H8mm" H 4850 3300 50  0001 C CNN
+F 2 "Button_Switch_THT:Push_E-Switch_KS01Q01" H 4850 3300 50  0001 C CNN
 F 3 "" H 4850 3300 50  0001 C CNN
 	1    4850 3100
@@
 F 0 "SW8" V 8450 3200 50  0000 L CNN
 F 1 "SW_Push" V 8350 3350 50  0000 C CNN
-F 2 "Button_Switch_THT:SW_PUSH_6mm_H8mm" H 8500 3300 50  0001 C CNN
+F 2 "Button_Switch_THT:Push_E-Switch_KS01Q01" H 8500 3300 50  0001 C CNN
 F 3 "" H 8500 3300 50  0001 C CNN
 	1    8500 3100
@@
 F 0 "SW7" V 8400 1150 50  0000 L CNN
 F 1 "SW_Push" V 8300 1300 50  0000 C CNN
-F 2 "Button_Switch_THT:SW_PUSH_6mm_H8mm" H 8450 1250 50  0001 C CNN
+F 2 "Button_Switch_THT:Push_E-Switch_KS01Q01" H 8450 1250 50  0001 C CNN
 F 3 "" H 8450 1250 50  0001 C CNN
 	1    8450 1050
@@
 F 0 "SW5" V 4850 1150 50  0000 L CNN
 F 1 "SW_Push" V 4750 1300 50  0000 C CNN
-F 2 "Button_Switch_THT:SW_PUSH_6mm_H8mm" H 4900 1250 50  0001 C CNN
+F 2 "Button_Switch_THT:Push_E-Switch_KS01Q01" H 4900 1250 50  0001 C CNN
 F 3 "" H 4900 1250 50  0001 C CNN
 	1    4900 1050
@@
 F 0 "SW1" V 1150 1150 50  0000 L CNN
 F 1 "SW_Push" V 1050 1300 50  0000 C CNN
-F 2 "Button_Switch_THT:SW_PUSH_6mm_H8mm" H 1200 1250 50  0001 C CNN
+F 2 "Button_Switch_THT:Push_E-Switch_KS01Q01" H 1200 1250 50  0001 C CNN
 F 3 "" H 1200 1250 50  0001 C CNN
 	1    1200 1050
@@
 F 0 "SW3" V 1200 5100 50  0000 L CNN
 F 1 "SW_Push" V 1100 5250 50  0000 C CNN
-F 2 "Button_Switch_THT:SW_PUSH_6mm_H8mm" H 1250 5200 50  0001 C CNN
+F 2 "Button_Switch_THT:Push_E-Switch_KS01Q01" H 1250 5200 50  0001 C CNN
 F 3 "" H 1250 5200 50  0001 C CNN
 	1    1250 5000
@@
 F 0 "SW6" V 4900 5100 50  0000 L CNN
 F 1 "SW_Push" V 4800 5250 50  0000 C CNN
-F 2 "Button_Switch_THT:SW_PUSH_6mm_H8mm" H 4950 5200 50  0001 C CNN
+F 2 "Button_Switch_THT:Push_E-Switch_KS01Q01" H 4950 5200 50  0001 C CNN
 F 3 "" H 4950 5200 50  0001 C CNN
 	1    4950 5000
@@
 F 0 "SW9" V 8450 5100 50  0000 L CNN
 F 1 "SW_Push" V 8350 5250 50  0000 C CNN
-F 2 "Button_Switch_THT:SW_PUSH_6mm_H8mm" H 8500 5200 50  0001 C CNN
+F 2 "Button_Switch_THT:Push_E-Switch_KS01Q01" H 8500 5200 50  0001 C CNN
 F 3 "" H 8500 5200 50  0001 C CNN
 	1    8500 5000

Commit message: Changed to horizontal resistors on PCB.
This resulted in only two vias, so that's nice.
Parts:
- R1, R10, R11, R12, R16, R17, R18, R2, R25, R26, R27, R3, R4, R5, R6, R7, R8, R9: footprint Resistor_THT:R_Axial_DIN0204_L3.6mm_D1.6mm_P1.90mm_Vertical -> Resistor_THT:R_Axial_DIN0207_L6.3mm_D2.5mm_P7.62mm_Horizontal
Changed lines of the file:
@@
 F 0 "R7" V 3200 900 50  0000 L CNN
 F 1 "1K" V 3200 700 50  0000 L CNN
-F 2 "Resistor_THT:R_Axial_DIN0204_L3.6mm_D1.6mm_P1.90mm_Vertical" H 3300 850 50  0001 C CNN
+F 2 "Resistor_THT:R_Axial_DIN0207_L6.3mm_D2.5mm_P7.62mm_Horizontal" H 3300 850 50  0001 C CNN
 F 3 "" H 3300 850 50  0001 C CNN
 	1    3300 850
@@
 F 0 "R16" V 6900 900 50  0000 L CNN
 F 1 "1K" V 6900 700 50  0000 L CNN
-F 2 "Resistor_THT:R_Axial_DIN0204_L3.6mm_D1.6mm_P1.90mm_Vertical" H 7000 850 50  0001 C CNN
+F 2 "Resistor_THT:R_Axial_DIN0207_L6.3mm_D2.5mm_P7.62mm_Horizontal" H 7000 850 50  0001 C CNN
 F 3 "" H 7000 850 50  0001 C CNN
 	1    7000 850
@@
 F 0 "R25" V 10450 900 50  0000 L CNN
 F 1 "1K" V 10450 700 50  0000 L CNN
-F 2 "Resistor_THT:R_Axial_DIN0204_L3.6mm_D1.6mm_P1.90mm_Vertical" H 10550 850 50  0001 C CNN
+F 2 "Resistor_THT:R_Axial_DIN0207_L6.3mm_D2.5mm_P7.62mm_Horizontal" H 10550 850 50  0001 C CNN
 F 3 "" H 10550 850 50  0001 C CNN
 	1    10550 850
@@
 F 0 "R3" H 1350 3600 50  0000 L CNN
 F 1 "1K" H 1350 3500 50  0000 L CNN
-F 2 "Resistor_THT:R_Axial_DIN0204_L3.6mm_D1.6mm_P1.90mm_Vertical" H 1250 3550 50  0001 C CNN
+F 2 "Resistor_THT:R_Axial_DIN0207_L6.3mm_D2.5mm_P7.62mm_Horizontal" H 1250 3550 50  0001 C CNN
 F 3 "" H 1250 3550 50  0001 C CNN
 	1    1250 3550
@@
 F 0 "R8" V 3250 2950 50  0000 L CNN
 F 1 "1K" V 3250 2750 50  0000 L CNN
-F 2 "Resistor_THT:R_Axial_DIN0204_L3.6mm_D1.6mm_P1.90mm_Vertical" H 3350 2900 50  0001 C CNN
+F 2 "Resistor_THT:R_Axial_DIN0207_L6.3mm_D2.5mm_P7.62mm_Horizontal" H 3350 2900 50  0001 C CNN
 F 3 "" H 3350 2900 50  0001 C CNN
 	1    3350 2900
@@
 F 0 "R17" V 6950 2950 50  0000 L CNN
 F 1 "1K" V 6950 2750 50  0000 L CNN
-F 2 "Resistor_THT:R_Axial_DIN0204_L3.6mm_D1.6mm_P1.90mm_Vertical" H 7050 2900 50  0001 C CNN
+F 2 "Resistor_THT:R_Axial_DIN0207_L6.3mm_D2.5mm_P7.62mm_Horizontal" H 7050 2900 50  0001 C CNN
 F 3 "" H 7050 2900 50  0001 C CNN
 	1    7050 2900
@@
 F 0 "R26" V 10500 2950 50  0000 L CNN
 F 1 "1K" V 10500 2750 50  0000 L CNN
-F 2 "Resistor_THT:R_Axial_DIN0204_L3.6mm_D1.6mm_P1.90mm_Vertical" H 10600 2900 50  0001 C CNN
+F 2 "Resistor_THT:R_Axial_DIN0207_L6.3mm_D2.5mm_P7.62mm_Horizontal" H 10600 2900 50  0001 C CNN
 F 3 "" H 10600 2900 50  0001 C CNN
 	1    10600 2900
@@
 F 0 "R9" V 3250 4850 50  0000 L CNN
 F 1 "1K" V 3250 4650 50  0000 L CNN
-F 2 "Resistor_THT:R_Axial_DIN0204_L3.6mm_D1.6mm_P1.90mm_Vertical" H 3350 4800 50  0001 C CNN
+F 2 "Resistor_THT:R_Axial_DIN0207_L6.3mm_D2.5mm_P7.62mm_Horizontal" H 3350 4800 50  0001 C CNN
 F 3 "" H 3350 4800 50  0001 C CNN
 	1    3350 4800
@@
 F 0 "R18" V 6950 4850 50  0000 L CNN
 F 1 "1K" V 6950 4650 50  0000 L CNN
-F 2 "Resistor_THT:R_Axial_DIN0204_L3.6mm_D1.6mm_P1.90mm_Vertical" H 7050 4800 50  0001 C CNN
+F 2 "Resistor_THT:R_Axial_DIN0207_L6.3mm_D2.5mm_P7.62mm_Horizontal" H 7050 4800 50  0001 C CNN
 F 3 "" H 7050 4800 50  0001 C CNN
 	1    7050 4800
@@
 F 0 "R27" V 10500 4850 50  0000 L CNN
 F 1 "1K" V 10500 4650 50  0000 L CNN
-F 2 "Resistor_THT:R_Axial_DIN0204_L3.6mm_D1.6mm_P1.90mm_Vertical" H 10600 4800 50  0001 C CNN
+F 2 "Resistor_THT:R_Axial_DIN0207_L6.3mm_D2.5mm_P7.62mm_Horizontal" H 10600 4800 50  0001 C CNN
 F 3 "" H 10600 4800 50  0001 C CNN
 	1    10600 4800
@@
 F 0 "R4" H 4950 3600 50  0000 L CNN
 F 1 "1K" H 4950 3500 50  0000 L CNN
-F 2 "Resistor_THT:R_Axial_DIN0204_L3.6mm_D1.6mm_P1.90mm_Vertical" H 4850 3550 50  0001 C CNN
+F 2 "Resistor_THT:R_Axial_DIN0207_L6.3mm_D2.5mm_P7.62mm_Horizontal" H 4850 3550 50  0001 C CNN
 F 3 "" H 4850 3550 50  0001 C CNN
 	1    4850 3550
@@
 F 0 "R11" H 8600 3600 50  0000 L CNN
 F 1 "1K" H 8600 3500 50  0000 L CNN
-F 2 "Resistor_THT:R_Axial_DIN0204_L3.6mm_D1.6mm_P1.90mm_Vertical" H 8500 3550 50  0001 C CNN
+F 2 "Resistor_THT:R_Axial_DIN0207_L6.3mm_D2.5mm_P7.62mm_Horizontal" H 8500 3550 50  0001 C CNN
 F 3 "" H 8500 3550 50  0001 C CNN
 	1    8500 3550
@@
 F 0 "R10" H 8550 1550 50  0000 L CNN
 F 1 "1K" H 8550 1450 50  0000 L CNN
-F 2 "Resistor_THT:R_Axial_DIN0204_L3.6mm_D1.6mm_P1.90mm_Vertical" H 8450 1500 50  0001 C CNN
+F 2 "Resistor_THT:R_Axial_DIN0207_L6.3mm_D2.5mm_P7.62mm_Horizontal" H 8450 1500 50  0001 C CNN
 F 3 "" H 8450 1500 50  0001 C CNN
 	1    8450 1500
@@
 F 0 "R5" H 5000 1550 50  0000 L CNN
 F 1 "1K" H 5000 1450 50  0000 L CNN
-F 2 "Resistor_THT:R_Axial_DIN0204_L3.6mm_D1.6mm_P1.90mm_Vertical" H 4900 1500 50  0001 C CNN
+F 2 "Resistor_THT:R_Axial_DIN0207_L6.3mm_D2.5mm_P7.62mm_Horizontal" H 4900 1500 50  0001 C CNN
 F 3 "" H 4900 1500 50  0001 C CNN
 	1    4900 1500
@@
 F 0 "R1" H 1300 1550 50  0000 L CNN
 F 1 "1K" H 1300 1450 50  0000 L CNN
-F 2 "Resistor_THT:R_Axial_DIN0204_L3.6mm_D1.6mm_P1.90mm_Vertical" H 1200 1500 50  0001 C CNN
+F 2 "Resistor_THT:R_Axial_DIN0207_L6.3mm_D2.5mm_P7.62mm_Horizontal" H 1200 1500 50  0001 C CNN
 F 3 "" H 1200 1500 50  0001 C CNN
 	1    1200 1500
@@
 F 0 "R2" H 1350 5500 50  0000 L CNN
 F 1 "1K" H 1350 5400 50  0000 L CNN
-F 2 "Resistor_THT:R_Axial_DIN0204_L3.6mm_D1.6mm_P1.90mm_Vertical" H 1250 5450 50  0001 C CNN
+F 2 "Resistor_THT:R_Axial_DIN0207_L6.3mm_D2.5mm_P7.62mm_Horizontal" H 1250 5450 50  0001 C CNN
 F 3 "" H 1250 5450 50  0001 C CNN
 	1    1250 5450
@@
 F 0 "R6" H 5050 5500 50  0000 L CNN
 F 1 "1K" H 5050 5400 50  0000 L CNN
-F 2 "Resistor_THT:R_Axial_DIN0204_L3.6mm_D1.6mm_P1.90mm_Vertical" H 4950 5450 50  0001 C CNN
+F 2 "Resistor_THT:R_Axial_DIN0207_L6.3mm_D2.5mm_P7.62mm_Horizontal" H 4950 5450 50  0001 C CNN
 F 3 "" H 4950 5450 50  0001 C CNN
 	1    4950 5450
@@
 F 0 "R12" H 8600 5500 50  0000 L CNN
 F 1 "1K" H 8600 5400 50  0000 L CNN
-F 2 "Resistor_THT:R_Axial_DIN0204_L3.6mm_D1.6mm_P1.90mm_Vertical" H 8500 5450 50  0001 C CNN
+F 2 "Resistor_THT:R_Axial_DIN0207_L6.3mm_D2.5mm_P7.62mm_Horizontal" H 8500 5450 50  0001 C CNN
 F 3 "" H 8500 5450 50  0001 C CNN
 	1    8500 5450
